Commit message: gazebo is loading

File: src/mobilebot/urdf/links.xacro (robot description, xacro)
@@ -6,11 +6,11 @@
             <origin rpy="0 0 0" xyz="0 0 0"/>
             <geometry>
-                <mesh filename="package://mobilebot/meshes/body.obj" scale="0.01 0.01 0.01"/>
-            </geometry>
-        </visual>
-        <collision>
-            <origin rpy="0 0 0" xyz="0 0 0"/>
-            <geometry>
-                <mesh filename="package://mobilebot/meshes/body.stl" scale="0.01 0.01 0.01"/>
+                <mesh filename="file://$(find mobilebot)/meshes/body.obj" scale="0.01 0.01 0.01"/>
+            </geometry>
+        </visual>
+        <collision>
+            <origin rpy="0 0 0" xyz="0 0 0"/>
+            <geometry>
+                <mesh filename="file://$(find mobilebot)/meshes/body.stl" scale="0.01 0.01 0.01"/>
             </geometry>
         </collision>
@@ -25,11 +25,11 @@
             <origin rpy="0 0 0" xyz="0 0 0"/>
             <geometry>
-                <mesh filename="package://mobilebot/meshes/wheel_left_side.obj" scale="0.01 0.01 0.01"/>
-            </geometry>
-        </visual>
-        <collision>
-            <origin rpy="0 0 0" xyz="0 0 0"/>
-            <geometry>
-                <mesh filename="package://mobilebot/meshes/wheel_left_side.stl" scale="0.01 0.01 0.01"/>
+                <mesh filename="file://$(find mobilebot)/meshes/wheel_left_side.obj" scale="0.01 0.01 0.01"/>
+            </geometry>
+        </visual>
+        <collision>
+            <origin rpy="0 0 0" xyz="0 0 0"/>
+            <geometry>
+                <mesh filename="file://$(find mobilebot)/meshes/wheel_left_side.stl" scale="0.01 0.01 0.01"/>
             </geometry>
         </collision>
@@ -44,11 +44,11 @@
             <origin rpy="0 0 0" xyz="0 0 0"/>
             <geometry>
-                <mesh filename="package://mobilebot/meshes/wheel_right_side.obj" scale="0.01 0.01 0.01"/>
-            </geometry>
-        </visual>
-        <collision>
-            <origin rpy="0 0 0" xyz="0 0 0"/>
-            <geometry>
-                <mesh filename="package://mobilebot/meshes/wheel_right_side.stl" scale="0.01 0.01 0.01"/>
+                <mesh filename="file://$(find mobilebot)/meshes/wheel_right_side.obj" scale="0.01 0.01 0.01"/>
+            </geometry>
+        </visual>
+        <collision>
+            <origin rpy="0 0 0" xyz="0 0 0"/>
+            <geometry>
+                <mesh filename="file://$(find mobilebot)/meshes/wheel_right_side.stl" scale="0.01 0.01 0.01"/>
             </geometry>
         </collision>
@@ -63,11 +63,11 @@
             <origin rpy="0 0 0" xyz="0 0 0"/>
             <geometry>
-                <mesh filename="package://mobilebot/meshes/wheel_right_side.obj" scale="0.01 0.01 0.01"/>
-            </geometry>
-        </visual>
-        <collision>
-            <origin rpy="0 0 0" xyz="0 0 0"/>
-            <geometry>
-                <mesh filename="package://mobilebot/meshes/wheel_right_side.stl" scale="0.01 0.01 0.01"/>
+                <mesh filename="file://$(find mobilebot)/meshes/wheel_right_side.obj" scale="0.01 0.01 0.01"/>
+            </geometry>
+        </visual>
+        <collision>
+            <origin rpy="0 0 0" xyz="0 0 0"/>
+            <geometry>
+                <mesh filename="file://$(find mobilebot)/meshes/wheel_right_side.stl" scale="0.01 0.01 0.01"/>
             </geometry>
         </collision>
@@ -82,11 +82,11 @@
             <origin rpy="0 0 0" xyz="0 0 0"/>
             <geometry>
-                <mesh filename="package://mobilebot/meshes/wheel_left_side.obj" scale="0.01 0.01 0.01"/>
-            </geometry>
-        </visual>
-        <collision>
-            <origin rpy="0 0 0" xyz="0 0 0"/>
-            <geometry>
-                <mesh filename="package://mobilebot/meshes/wheel_left_side.stl" scale="0.01 0.01 0.01"/>
+                <mesh filename="file://$(find mobilebot)/meshes/wheel_left_side.obj" scale="0.01 0.01 0.01"/>
+            </geometry>
+        </visual>
+        <collision>
+            <origin rpy="0 0 0" xyz="0 0 0"/>
+            <geometry>
+                <mesh filename="file://$(find mobilebot)/meshes/wheel_left_side.stl" scale="0.01 0.01 0.01"/>
             </geometry>
         </collision>
@@ -101,11 +101,11 @@
             <origin rpy="0 0 0" xyz="0 0 0"/>
             <geometry>
-                <mesh filename="package://mobilebot/meshes/Base.obj" scale="0.01 0.01 0.01"/>
-            </geometry>
-        </visual>
-        <collision>
-            <origin rpy="0 0 0" xyz="0 0 0"/>
-            <geometry>
-                <mesh filename="package://mobilebot/meshes/Base.stl" scale="0.01 0.01 0.01"/>
+                <mesh filename="file://$(find mobilebot)/meshes/Base.obj" scale="0.01 0.01 0.01"/>
+            </geometry>
+        </visual>
+        <collision>
+            <origin rpy="0 0 0" xyz="0 0 0"/>
+            <geometry>
+                <mesh filename="file://$(find mobilebot)/meshes/Base.stl" scale="0.01 0.01 0.01"/>
             </geometry>
         </collision>
@@ -120,11 +120,11 @@
             <origin rpy="0 0 0" xyz="0 0 0"/>
             <geometry>
-                <mesh filename="package://mobilebot/meshes/Shoulder.obj" scale="0.01 0.01 0.01"/>
-            </geometry>
-        </visual>
-        <collision>
-            <origin rpy="0 0 0" xyz="0 0 0"/>
-            <geometry>
-                <mesh filename="package://mobilebot/meshes/Shoulder.stl" scale="0.01 0.01 0.01"/>
+                <mesh filename="file://$(find mobilebot)/meshes/Shoulder.obj" scale="0.01 0.01 0.01"/>
+            </geometry>
+        </visual>
+        <collision>
+            <origin rpy="0 0 0" xyz="0 0 0"/>
+            <geometry>
+                <mesh filename="file://$(find mobilebot)/meshes/Shoulder.stl" scale="0.01 0.01 0.01"/>
             </geometry>
         </collision>
@@ -139,11 +139,11 @@
             <origin rpy="0 0 0" xyz="0 0 0"/>
             <geometry>
-                <mesh filename="package://mobilebot/meshes/Link.obj" scale="0.01 0.01 0.01"/>
-            </geometry>
-        </visual>
-        <collision>
-            <origin rpy="0 0 0" xyz="0 0 0"/>
-            <geometry>
-                <mesh filename="package://mobilebot/meshes/Link.stl" scale="0.01 0.01 0.01"/>
+                <mesh filename="file://$(find mobilebot)/meshes/Link.obj" scale="0.01 0.01 0.01"/>
+            </geometry>
+        </visual>
+        <collision>
+            <origin rpy="0 0 0" xyz="0 0 0"/>
+            <geometry>
+                <mesh filename="file://$(find mobilebot)/meshes/Link.stl" scale="0.01 0.01 0.01"/>
             </geometry>
         </collision>
@@ -158,11 +158,11 @@
             <origin rpy="0 0 0" xyz="0 0 0"/>
             <geometry>
-                <mesh filename="package://mobilebot/meshes/Elbow.obj" scale="0.01 0.01 0.01"/>
-            </geometry>
-        </visual>
-        <collision>
-            <origin rpy="0 0 0" xyz="0 0 0"/>
-            <geometry>
-                <mesh filename="package://mobilebot/meshes/Elbow.stl" scale="0.01 0.01 0.01"/>
+                <mesh filename="file://$(find mobilebot)/meshes/Elbow.obj" scale="0.01 0.01 0.01"/>
+            </geometry>
+        </visual>
+        <collision>
+            <origin rpy="0 0 0" xyz="0 0 0"/>
+            <geometry>
+                <mesh filename="file://$(find mobilebot)/meshes/Elbow.stl" scale="0.01 0.01 0.01"/>
             </geometry>
         </collision>
@@ -177,11 +177,11 @@
             <origin rpy="0 0 0" xyz="0 0 0"/>
             <geometry>
-                <mesh filename="package://mobilebot/meshes/Wrist.obj" scale="0.01 0.01 0.01"/>
-            </geometry>
-        </visual>
-        <collision>
-            <origin rpy="0 0 0" xyz="0 0 0"/>
-            <geometry>
-                <mesh filename="package://mobilebot/meshes/Wrist.stl" scale="0.01 0.01 0.01"/>
+                <mesh filename="file://$(find mobilebot)/meshes/Wrist.obj" scale="0.01 0.01 0.01"/>
+            </geometry>
+        </visual>
+        <collision>
+            <origin rpy="0 0 0" xyz="0 0 0"/>
+            <geometry>
+                <mesh filename="file://$(find mobilebot)/meshes/Wrist.stl" scale="0.01 0.01 0.01"/>
             </geometry>
         </collision>
@@ -196,11 +196,11 @@
             <origin rpy="0 0 0" xyz="0 0 0"/>
             <geometry>
-                <mesh filename="package://mobilebot/meshes/Gripper.obj" scale="0.01 0.01 0.01"/>
-            </geometry>
-        </visual>
-        <collision>
-            <origin rpy="0 0 0" xyz="0 0 0"/>
-            <geometry>
-                <mesh filename="package://mobilebot/meshes/Gripper.stl" scale="0.01 0.01 0.01"/>
+                <mesh filename="file://$(find mobilebot)/meshes/Gripper.obj" scale="0.01 0.01 0.01"/>
+            </geometry>
+        </visual>
+        <collision>
+            <origin rpy="0 0 0" xyz="0 0 0"/>
+            <geometry>
+                <mesh filename="file://$(find mobilebot)/meshes/Gripper.stl" scale="0.01 0.01 0.01"/>
             </geometry>
         </collision>
