Commit message: updating

File: install/mobilebot/share/mobilebot/urdf/gazebo.xacro (robot description, xacro)
@@ -1 +1,35 @@
-/home/hars22/rosws/src/mobilebot/urdf/gazebo.xacro
+<?xml version="1.0"?>
+<robot name="Robot" xmlns:xacro="http://ros.org/wiki/xacro">
+    <gazebo>
+        <plugin filename="libgz_ros2_control-system.so" name="gz_ros2_control::GazeboSimROS2ControlPlugin">
+            <robot_param>robot_description</robot_param>
+            <robot_param_node>robot_state_publisher</robot_param_node>
+            <parameters>/home/hars22/rosws/src/mobilebot_controller/config/mobilebot_controller.yaml</parameters>
+        </plugin>
+    </gazebo>
+    <gazebo reference="lidar_link">
+        <sensor type="ray" name="lidar">
+            <update_rate>10</update_rate>
+            <ray>
+            <scan>
+                <horizontal>
+                <samples>720</samples>
+                <resolution>1</resolution>
+                <min_angle>-1.5708</min_angle>
+                <max_angle>1.5708</max_angle>
+                </horizontal>
+            </scan>
+            <range>
+                <min>0.12</min>
+                <max>8.0</max>
+                <resolution>0.01</resolution>
+            </range>
+            </ray>
+            <!-- ROS 2 plugin for Ignition/Fortress -->
+            <plugin name="ros2_laser" filename="gz-sim-ros2-ray-sensor-system">
+            <topic>lidar_scan</topic>
+            <frame_name>lidar_link</frame_name>
+            </plugin>
+        </sensor>
+    </gazebo>
+</robot>

File: install/mobilebot/share/mobilebot/urdf/joints.xacro (robot description, xacro)
@@ -1 +1,81 @@
-/home/hars22/rosws/src/mobilebot/urdf/joints.xacro
+<?xml version="1.0"?>
+<robot name="Robot" xmlns:xacro="http://ros.org/wiki/xacro">
+    <joint name="virtual_joint" type="fixed">
+        <parent link="base_link"/>
+        <child link="mobile_robot_body"/>
+        <origin rpy="0 0 0" xyz="0 0 0.0975"/>
+    </joint>
+    <joint name="caster_wheel_left_joint" type="continuous">
+        <parent link="mobile_robot_body"/>
+        <child link="caster_wheel_left"/>
+        <axis xyz="1 0 0"/>
+        <origin rpy="0 0 0" xyz="0.475 -0.2275 0.065"/>
+        <limit effort="30.0" velocity="10.0"/>
+    </joint>
+    <joint name="caster_wheel_right_joint" type="continuous">
+        <parent link="mobile_robot_body"/>
+        <child link="caster_wheel_right"/>
+        <axis xyz="1 0 0"/>
+        <origin rpy="0 0 0" xyz="-0.475 -0.2275 0.065"/>
+        <limit effort="30.0" velocity="10.0"/>
+    </joint>
+    <joint name="driver_wheel_right_joint" type="continuous">
+        <parent link="mobile_robot_body"/>
+        <child link="driver_wheel_right"/>
+        <axis xyz="1 0 0"/>
+        <origin rpy="0 0 0" xyz="-0.475 0.2275 0.065"/>
+        <limit effort="30.0" velocity="10.0"/>
+    </joint>
+    <joint name="driver_wheel_left_joint" type="continuous">
+        <parent link="mobile_robot_body"/>
+        <child link="driver_wheel_left"/>
+        <axis xyz="1 0 0"/>
+        <origin rpy="0 0 0" xyz="0.475 0.2275 0.065"/>
+        <limit effort="30.0" velocity="10.0"/>
+    </joint>
+    <joint name="manipulator_base_mobile_joint" type="fixed">
+        <parent link="mobile_robot_body"/>
+        <child link="manipulator_base"/>
+        <origin rpy="0 0 0" xyz="0 -0.1 0.13"/>
+    </joint>
+    <joint name="manipulator_base_shoulder_joint" type="revolute">
+        <parent link="manipulator_base"/>
+        <child link="manipulator_shoulder"/>
+        <axis xyz="0 0 1"/>
+        <origin rpy="0 0 0" xyz="0 0 0.17"/>
+        <limit lower="-1.57" upper="1.57" effort="30.0" velocity="10.0"/>
+    </joint>
+    <joint name="manipulator_shoulder_link_joint" type="revolute">
+        <parent link="manipulator_shoulder"/>
+        <child link="manipulator_link"/>
+        <axis xyz="1 0 0"/>
+        <origin rpy="0 0 0" xyz="0 0 0.336"/>
+        <limit lower="-1.57" upper="1.57" effort="30.0" velocity="10.0"/>
+    </joint>
+    <joint name="manipulator_link_elbow_joint" type="revolute">
+        <parent link="manipulator_link"/>
+        <child link="manipulator_elbow"/>
+        <axis xyz="1 0 0"/>
+        <origin rpy="0 0 0" xyz="0 0 0.5"/>
+        <limit lower="-1.57" upper="1.57" effort="30.0" velocity="10.0"/>
+    </joint>
+    <joint name="manipulator_elbow_wrist_joint" type="revolute">
+        <parent link="manipulator_elbow"/>
+        <child link="manipulator_wrist"/>
+        <axis xyz="1 0 0"/>
+        <origin rpy="0 0 0" xyz="0 -0.427455 0.145"/>
+        <limit lower="-1.57" upper="1.57" effort="30.0" velocity="10.0"/>
+    </joint>
+    <joint name="manipulator_wrist_gripper_joint" type="revolute">
+        <parent link="manipulator_wrist"/>
+        <child link="manipulator_gripper"/>
+        <axis xyz="0 1 0"/>
+        <origin rpy="0 0 0" xyz="0 -0.105 0"/>
+        <limit lower="-1.57" upper="1.57" effort="30.0" velocity="10.0"/>
+    </joint>
+    <joint name="lidar_joint" type="fixed">
+        <parent link="mobile_robot_body"/>
+        <child link="lidar_link"/>
+        <origin xyz="0 0.3 0.13" rpy="0 0 0"/>
+    </joint>
+</robot>

File: install/mobilebot/share/mobilebot/urdf/links.xacro (robot description, xacro)
@@ -1 +1,237 @@
-/home/hars22/rosws/src/mobilebot/urdf/links.xacro
+<?xml version="1.0"?>
+<robot name="Robot" xmlns:xacro="http://ros.org/wiki/xacro">
+    <link name="base_link"/>
+    <link name="mobile_robot_body">
+        <visual>
+            <origin rpy="0 0 0" xyz="0 0 0"/>
+            <geometry>
+                <mesh filename="file://$(find mobilebot)/meshes/body.obj" scale="0.01 0.01 0.01"/>
+            </geometry>
+        </visual>
+        <collision>
+            <origin rpy="0 0 0" xyz="0 0 0"/>
+            <geometry>
+                <mesh filename="file://$(find mobilebot)/meshes/body.stl" scale="0.01 0.01 0.01"/>
+            </geometry>
+        </collision>
+        <inertial>
+            <origin xyz="0 0 0.05" rpy="0 0 0"/>
+            <mass value="10.0"/>
+            <inertia ixx="0.04" ixy="0" ixz="0" iyy="0.04" iyz="0" izz="0.06"/>
+        </inertial>
+    </link>
+    <link name="caster_wheel_left">
+        <visual>
+            <origin rpy="0 0 0" xyz="0 0 0"/>
+            <geometry>
+                <mesh filename="file://$(find mobilebot)/meshes/wheel_left_side.obj" scale="0.01 0.01 0.01"/>
+            </geometry>
+        </visual>
+        <collision>
+            <origin rpy="0 0 0" xyz="0 0 0"/>
+            <geometry>
+                <mesh filename="file://$(find mobilebot)/meshes/wheel_left_side.stl" scale="0.01 0.01 0.01"/>
+            </geometry>
+        </collision>
+        <inertial>
+            <origin xyz="0 0 0" rpy="0 0 0"/>
+            <mass value="1"/> <!-- kg -->
+            <inertia ixx="0.0002" ixy="0" ixz="0" iyy="0.0002" iyz="0" izz="0.0001"/>
+        </inertial>
+    </link>
+    <link name="caster_wheel_right">
+        <visual>
+            <origin rpy="0 0 0" xyz="0 0 0"/>
+            <geometry>
+                <mesh filename="file://$(find mobilebot)/meshes/wheel_right_side.obj" scale="0.01 0.01 0.01"/>
+            </geometry>
+        </visual>
+        <collision>
+            <origin rpy="0 0 0" xyz="0 0 0"/>
+            <geometry>
+                <mesh filename="file://$(find mobilebot)/meshes/wheel_right_side.stl" scale="0.01 0.01 0.01"/>
+            </geometry>
+        </collision>
+        <inertial>
+            <origin xyz="0 0 0" rpy="0 0 0"/>
+            <mass value="1"/> <!-- kg -->
+            <inertia ixx="0.0002" ixy="0" ixz="0" iyy="0.0002" iyz="0" izz="0.0001"/>
+        </inertial>
+    </link>
+    <link name="driver_wheel_right">
+        <visual>
+            <origin rpy="0 0 0" xyz="0 0 0"/>
+            <geometry>
+                <mesh filename="file://$(find mobilebot)/meshes/wheel_right_side.obj" scale="0.01 0.01 0.01"/>
+            </geometry>
+        </visual>
+        <collision>
+            <origin rpy="0 0 0" xyz="0 0 0"/>
+            <geometry>
+                <mesh filename="file://$(find mobilebot)/meshes/wheel_right_side.stl" scale="0.01 0.01 0.01"/>
+            </geometry>
+        </collision>
+        <inertial>
+            <origin xyz="0 0 0" rpy="0 0 0"/>
+            <mass value="1"/> <!-- kg -->
+            <inertia ixx="0.0002" ixy="0" ixz="0" iyy="0.0002" iyz="0" izz="0.0001"/>
+        </inertial>
+    </link>
+    <link name="driver_wheel_left">
+        <visual>
+            <origin rpy="0 0 0" xyz="0 0 0"/>
+            <geometry>
+                <mesh filename="file://$(find mobilebot)/meshes/wheel_left_side.obj" scale="0.01 0.01 0.01"/>
+            </geometry>
+        </visual>
+        <collision>
+            <origin rpy="0 0 0" xyz="0 0 0"/>
+            <geometry>
+                <mesh filename="file://$(find mobilebot)/meshes/wheel_left_side.stl" scale="0.01 0.01 0.01"/>
+            </geometry>
+        </collision>
+        <inertial>
+            <origin xyz="0 0 0" rpy="0 0 0"/>
+            <mass value="1"/> <!-- kg -->
+            <inertia ixx="0.0002" ixy="0" ixz="0" iyy="0.0002" iyz="0" izz="0.0001"/>
+        </inertial>
+    </link>
+    <link name="manipulator_base">
+        <visual>
+            <origin rpy="0 0 0" xyz="0 0 0"/>
+            <geometry>
+                <mesh filename="file://$(find mobilebot)/meshes/Base.obj" scale="0.01 0.01 0.01"/>
+            </geometry>
+        </visual>
+        <collision>
+            <origin rpy="0 0 0" xyz="0 0 0"/>
+            <geometry>
+                <mesh filename="file://$(find mobilebot)/meshes/Base.stl" scale="0.01 0.01 0.01"/>
+            </geometry>
+        </collision>
+        <inertial>
+            <origin xyz="0 0 0" rpy="0 0 0"/>
+            <mass value="1"/>
+            <inertia ixx="0.02" ixy="0" ixz="0" iyy="0.02" iyz="0" izz="0.03"/>
+        </inertial>
+    </link>
+    <link name="manipulator_shoulder">
+        <visual>
+            <origin rpy="0 0 0" xyz="0 0 0"/>
+            <geometry>
+                <mesh filename="file://$(find mobilebot)/meshes/Shoulder.obj" scale="0.01 0.01 0.01"/>
+            </geometry>
+        </visual>
+        <collision>
+            <origin rpy="0 0 0" xyz="0 0 0"/>
+            <geometry>
+                <mesh filename="file://$(find mobilebot)/meshes/Shoulder.stl" scale="0.01 0.01 0.01"/>
+            </geometry>
+        </collision>
+        <inertial>
+            <origin xyz="0 0 0.1" rpy="0 0 0"/>
+            <mass value="1.0"/>
+            <inertia ixx="0.005" ixy="0" ixz="0" iyy="0.005" iyz="0" izz="0.002"/>
+        </inertial>
+    </link>
+    <link name="manipulator_link">
+        <visual>
+            <origin rpy="0 0 0" xyz="0 0 0"/>
+            <geometry>
+                <mesh filename="file://$(find mobilebot)/meshes/Link.obj" scale="0.01 0.01 0.01"/>
+            </geometry>
+        </visual>
+        <collision>
+            <origin rpy="0 0 0" xyz="0 0 0"/>
+            <geometry>
+                <mesh filename="file://$(find mobilebot)/meshes/Link.stl" scale="0.01 0.01 0.01"/>
+            </geometry>
+        </collision>
+        <inertial>
+            <origin xyz="0 0 0.15" rpy="0 0 0"/>
+            <mass value="1.0"/>
+            <inertia ixx="0.003" ixy="0" ixz="0" iyy="0.003" iyz="0" izz="0.001"/>
+        </inertial>
+    </link>
+    <link name="manipulator_elbow">
+        <visual>
+            <origin rpy="0 0 0" xyz="0 0 0"/>
+            <geometry>
+                <mesh filename="file://$(find mobilebot)/meshes/Elbow.obj" scale="0.01 0.01 0.01"/>
+            </geometry>
+        </visual>
+        <collision>
+            <origin rpy="0 0 0" xyz="0 0 0"/>
+            <geometry>
+                <mesh filename="file://$(find mobilebot)/meshes/Elbow.stl" scale="0.01 0.01 0.01"/>
+            </geometry>
+        </collision>
+        <inertial>
+            <origin xyz="0 0 0.05" rpy="0 0 0"/>
+            <mass value="1.0"/>
+            <inertia ixx="0.002" ixy="0" ixz="0" iyy="0.002" iyz="0" izz="0.001"/>
+        </inertial>
+    </link>
+    <link name="manipulator_wrist">
+        <visual>
+            <origin rpy="0 0 0" xyz="0 0 0"/>
+            <geometry>
+                <mesh filename="file://$(find mobilebot)/meshes/Wrist.obj" scale="0.01 0.01 0.01"/>
+            </geometry>
+        </visual>
+        <collision>
+            <origin rpy="0 0 0" xyz="0 0 0"/>
+            <geometry>
+                <mesh filename="file://$(find mobilebot)/meshes/Wrist.stl" scale="0.01 0.01 0.01"/>
+            </geometry>
+        </collision>
+        <inertial>
+            <origin xyz="0 0 0.03" rpy="0 0 0"/>
+            <mass value="0.8"/>
+            <inertia ixx="0.0008" ixy="0" ixz="0" iyy="0.0008" iyz="0" izz="0.0005"/>
+        </inertial>
+    </link>
+    <link name="manipulator_gripper">
+        <visual>
+            <origin rpy="0 0 0" xyz="0 0 0"/>
+            <geometry>
+                <mesh filename="file://$(find mobilebot)/meshes/Gripper.obj" scale="0.01 0.01 0.01"/>
+            </geometry>
+        </visual>
+        <collision>
+            <origin rpy="0 0 0" xyz="0 0 0"/>
+            <geometry>
+                <mesh filename="file://$(find mobilebot)/meshes/Gripper.stl" scale="0.01 0.01 0.01"/>
+            </geometry>
+        </collision>
+        <inertial>
+            <origin xyz="0 0 0.02" rpy="0 0 0"/>
+            <mass value="0.5"/>
+            <inertia ixx="0.0005" ixy="0" ixz="0" iyy="0.0005" iyz="0" izz="0.0003"/>
+        </inertial>
+    </link>
+    <material name="black">
+        <color rgba="0 0 0 1"/>
+    </material>
+    <link name="lidar_link">
+        <visual>
+            <origin rpy="0 0 0" xyz="0 0 0"/>
+            <geometry>
+                <cylinder radius="0.1" length="0.075"/>
+            </geometry>
+            <material name="black"/>
+        </visual>
+        <collision>
+            <origin rpy="0 0 0" xyz="0 0 0"/>
+            <geometry>
+                <cylinder radius="0.1" length="0.075"/>
+            </geometry>
+        </collision>
+        <inertial>
+            <mass value="0.3"/>
+            <origin xyz="0 0 0" rpy="0 0 0"/>
+            <inertia ixx="0.001" iyy="0.001" izz="0.001"
+                    ixy="0.0" ixz="0.0" iyz="0.0"/>
+        </inertial>
+    </link>
+</robot>

File: install/mobilebot/share/mobilebot/urdf/robot.urdf.xacro (robot description, xacro)
@@ -1 +1,8 @@
-/home/hars22/rosws/src/mobilebot/urdf/robot.urdf.xacro
+<?xml version="1.0"?>
+<robot name="Robot" xmlns:xacro="http://ros.org/wiki/xacro">
+    <xacro:include filename="$(find mobilebot)/urdf/gazebo.xacro"/>
+    <xacro:include filename="$(find mobilebot)/urdf/ros2_control.xacro"/>
+    <xacro:include filename="$(find mobilebot)/urdf/transmission.xacro"/>]
+    <xacro:include filename="$(find mobilebot)/urdf/links.xacro"/>
+    <xacro:include filename="$(find mobilebot)/urdf/joints.xacro"/>
+</robot>

File: install/mobilebot/share/mobilebot/urdf/ros2_control.xacro (robot description, xacro)
@@ -1 +1,53 @@
-/home/hars22/rosws/src/mobilebot/urdf/ros2_control.xacro
+<?xml version="1.0"?>
+<robot name="Robot" xmlns:xacro="http://ros.org/wiki/xacro">
+    <ros2_control name="robotsystem" type="system">
+        <hardware>
+            <plugin>gz_ros2_control/GazeboSimSystem</plugin>
+        </hardware>
+        <joint name="manipulator_base_shoulder_joint">
+            <command_interface name="position">
+                <param name="min">-1.57</param>
+                <param name="max">1.57</param>
+            </command_interface>
+            <state_interface name="position"/>
+        </joint>
+        <joint name="manipulator_shoulder_link_joint">
+            <command_interface name="position">
+                <param name="min">-1.57</param>
+                <param name="max">1.57</param>
+            </command_interface>
+            <state_interface name="position"/>
+        </joint>
+        <joint name="manipulator_link_elbow_joint">
+            <command_interface name="position">
+                <param name="min">-1.57</param>
+                <param name="max">1.57</param>
+            </command_interface>
+            <state_interface name="position"/>
+        </joint>
+        <joint name="manipulator_elbow_wrist_joint">
+            <command_interface name="position">
+                <param name="min">-1.57</param>
+                <param name="max">1.57</param>
+            </command_interface>
+            <state_interface name="position"/>
+        </joint>
+        <joint name="manipulator_wrist_gripper_joint">
+            <command_interface name="position">
+                <param name="min">-1.57</param>
+                <param name="max">1.57</param>
+            </command_interface>
+            <state_interface name="position"/>
+        </joint>
+        <joint name="driver_wheel_left_joint">
+            <command_interface name="velocity"/>
+            <state_interface name="position"/>
+            <state_interface name="velocity"/>
+        </joint>
+        <joint name="driver_wheel_right_joint">
+            <command_interface name="velocity"/>
+            <state_interface name="position"/>
+            <state_interface name="velocity"/>
+        </joint>
+    </ros2_control>
+</robot>

File: install/mobilebot/share/mobilebot/urdf/transmission.xacro (robot description, xacro)
@@ -1 +1,93 @@
-/home/hars22/rosws/src/mobilebot/urdf/transmission.xacro
+<?xml version="1.0"?>
+<robot name="Robot" xmlns:xacro="http://ros.org/wiki/xacro">
+    <transmission name="transmission_1">
+        <type>transmission_interface/SimpleTransmission</type>
+        <joint name="manipulator_base_shoulder_joint">
+            <hardwareInterface>hardware_interface/PositionJointInterface</hardwareInterface>
+        </joint>
+        <actuator name="Base_Shoulder_actuator">
+            <mechanicalReduction>1.0</mechanicalReduction>
+            <hardwareInterface>hardware_interface/PositionJointInterface</hardwareInterface>
+        </actuator>
+    </transmission>
+    <transmission name="transmission_2">
+        <type>transmission_interface/SimpleTransmission</type>
+        <joint name="manipulator_shoulder_link_joint">
+            <hardwareInterface>hardware_interface/PositionJointInterface</hardwareInterface>
+        </joint>
+        <actuator name="shoulder_link_actuator">
+            <mechanicalReduction>1.0</mechanicalReduction>
+            <hardwareInterface>hardware_interface/PositionJointInterface</hardwareInterface>
+        </actuator>
+    </transmission>
+    <transmission name="transmission_3">
+        <type>transmission_interface/SimpleTransmission</type>
+        <joint name="manipulator_link_elbow_joint">
+            <hardwareInterface>hardware_interface/PositionJointInterface</hardwareInterface>
+        </joint>
+        <actuator name="link_elbow_actuator">
+            <mechanicalReduction>1.0</mechanicalReduction>
+            <hardwareInterface>hardware_interface/PositionJointInterface</hardwareInterface>
+        </actuator>
+    </transmission>
+    <transmission name="transmission_4">
+        <type>transmission_interface/SimpleTransmission</type>
+        <joint name="manipulator_elbow_wrist_joint">
+            <hardwareInterface>hardware_interface/PositionJointInterface</hardwareInterface>
+        </joint>
+        <actuator name="elbow_wrist_actuator">
+            <mechanicalReduction>1.0</mechanicalReduction>
+            <hardwareInterface>hardware_interface/PositionJointInterface</hardwareInterface>
+        </actuator>
+    </transmission>
+    <transmission name="transmission_5">
+        <type>transmission_interface/SimpleTransmission</type>
+        <joint name="manipulator_wrist_gripper_joint">
+            <hardwareInterface>hardware_interface/PositionJointInterface</hardwareInterface>
+        </joint>
+        <actuator name="wrist_gripper_actuator">
+            <mechanicalReduction>1.0</mechanicalReduction>
+            <hardwareInterface>hardware_interface/PositionJointInterface</hardwareInterface>
+        </actuator>
+    </transmission>
+    <transmission name="transmission_6">
+        <type>transmission_interface/SimpleTransmission</type>
+        <joint name="caster_wheel_left_joint">
+            <hardwareInterface>hardware_interface/PositionJointInterface</hardwareInterface>
+        </joint>
+        <actuator name="caster_wheel_left_actuator">
+            <mechanicalReduction>1.0</mechanicalReduction>
+            <hardwareInterface>hardware_interface/PositionJointInterface</hardwareInterface>
+        </actuator>
+    </transmission>
+    <transmission name="transmission_7">
+        <type>transmission_interface/SimpleTransmission</type>
+        <joint name="caster_wheel_right_joint">
+            <hardwareInterface>hardware_interface/PositionJointInterface</hardwareInterface>
+        </joint>
+        <actuator name="caster_wheel_right_actuator">
+            <mechanicalReduction>1.0</mechanicalReduction>
+            <hardwareInterface>hardware_interface/PositionJointInterface</hardwareInterface>
+        </actuator>
+    </transmission>
+    <transmission name="transmission_8">
+        <type>transmission_interface/SimpleTransmission</type>
+        <joint name="driver_wheel_right_joint">
+            <hardwareInterface>hardware_interface/VelocityJointInterface</hardwareInterface>
+        </joint>
+        <actuator name="driver_wheel_right_actuator">
+            <mechanicalReduction>1.0</mechanicalReduction>
+            <hardwareInterface>hardware_interface/VelocityJointInterface</hardwareInterface>
+        </actuator>
+    </transmission>
+    <transmission name="transmission_9">
+        <type>transmission_interface/SimpleTransmission</type>
+        <joint name="driver_wheel_left_joint">
+            <hardwareInterface>hardware_interface/VelocityJointInterface</hardwareInterface>
+        </joint>
+        <actuator name="driver_wheel_left_actuator">
+            <mechanicalReduction>1.0</mechanicalReduction>
+            <hardwareInterface>hardware_interface/VelocityJointInterface</hardwareInterface>
+        </actuator>
+    </transmission>
+</robot>

File: install/robot_description/share/robot_description/urdf/robot.urdf.xacro (robot description, xacro)
@@ -1 +1,8 @@
-/home/hars22/rosws/src/robot_description/urdf/robot.urdf.xacro
+<?xml version="1.0"?>
+<robot name="Robot" xmlns:xacro="http://ros.org/wiki/xacro">
+    <xacro:include filename="$(find robot_description)/urdf/gazebo.xacro"/>
+    <xacro:include filename="$(find robot_description)/urdf/ros2_control.xacro"/>
+    <xacro:include filename="$(find robot_description)/urdf/transmission.xacro"/>]
+    <xacro:include filename="$(find robot_description)/urdf/links.xacro"/>
+    <xacro:include filename="$(find robot_description)/urdf/joints.xacro"/>
+</robot>
