Commit message: updating

File: src/mobilebot/urdf/gazebo.xacro (robot description, xacro)
@@ -10,8 +10,5 @@
     <gazebo reference="lidar_link">
         <sensor type="ray" name="lidar">
-            <pose>0 0 0 0 0 0</pose>
-            <visualize>true</visualize>
-            <update_rate>10.0</update_rate>
-            <topic>/lidar_scan</topic>
+            <update_rate>10</update_rate>
             <ray>
             <scan>
@@ -29,4 +26,9 @@
             </range>
             </ray>
+            <!-- ROS 2 plugin for Ignition/Fortress -->
+            <plugin name="ros2_laser" filename="gz-sim-ros2-ray-sensor-system">
+            <topic>lidar_scan</topic>
+            <frame_name>lidar_link</frame_name>
+            </plugin>
         </sensor>
     </gazebo>

File: src/robot_description/urdf/robot.urdf.xacro (robot description, xacro)
@@ -1,286 +1,8 @@
 <?xml version="1.0"?>
-<robot xmlns:xacro="http://www.ros.org/wiki/xacro" name="Robot">
-    <link name="world"/>
-    <link name="base_link">
-        <visual>
-            <origin rpy="0 0 0" xyz="0 0 0"/>
-            <geometry>
-                <mesh filename="package://robot_description/meshes/body.stl" scale="0.01 0.01 0.01"/>
-            </geometry>
-        </visual>
-        <collision>
-            <origin rpy="0 0 0" xyz="0 0 0"/>
-            <geometry>
-                <mesh filename="package://robot_description/meshes/body.stl" scale="0.01 0.01 0.01"/>
-            </geometry>
-        </collision>
-        <inertial>
-            <origin xyz="0 0 0.05" rpy="0 0 0"/>
-            <mass value="5.0"/>
-            <inertia ixx="0.04" ixy="0" ixz="0" iyy="0.04" iyz="0" izz="0.06"/>
-        </inertial>
-    </link>
-    <joint name="virtual_joint" type="fixed">
-        <parent link="world"/>
-        <child link="base_link"/>
-        <origin rpy="0 0 0" xyz="0 0 0"/>
-    </joint>
-    <link name="caster_wheel_left">
-        <visual>
-            <origin rpy="0 0 0" xyz="0 0 0"/>
-            <geometry>
-                <mesh filename="package://robot_description/meshes/wheel_left_side.stl" scale="0.01 0.01 0.01"/>
-            </geometry>
-        </visual>
-        <collision>
-            <origin rpy="0 0 0" xyz="0 0 0"/>
-            <geometry>
-                <mesh filename="package://robot_description/meshes/wheel_left_side.stl" scale="0.01 0.01 0.01"/>
-            </geometry>
-        </collision>
-        <inertial>
-            <origin xyz="0 0 0" rpy="0 0 0"/>
-            <mass value="0.3"/> <!-- kg -->
-            <inertia ixx="0.0002" ixy="0" ixz="0" iyy="0.0002" iyz="0" izz="0.0001"/>
-        </inertial>
-    </link>
-    <joint name="caster_wheel_left_joint" type="revolute">
-        <parent link="base_link"/>
-        <child link="caster_wheel_left"/>
-        <axis xyz="1 0 0"/>
-        <origin rpy="0 0 0" xyz="4.75 -2.275 0.65"/>
-        <limit lower="-1.57" upper="1.57" effort="30.0" velocity="10.0"/>
-    </joint>
-    <link name="caster_wheel_right">
-        <visual>
-            <origin rpy="0 0 0" xyz="0 0 0"/>
-            <geometry>
-                <mesh filename="package://robot_description/meshes/wheel_right_side.stl" scale="0.01 0.01 0.01"/>
-            </geometry>
-        </visual>
-        <collision>
-            <origin rpy="0 0 0" xyz="0 0 0"/>
-            <geometry>
-                <mesh filename="package://robot_description/meshes/wheel_right_side.stl" scale="0.01 0.01 0.01"/>
-            </geometry>
-        </collision>
-        <inertial>
-            <origin xyz="0 0 0" rpy="0 0 0"/>
-            <mass value="0.3"/> <!-- kg -->
-            <inertia ixx="0.0002" ixy="0" ixz="0" iyy="0.0002" iyz="0" izz="0.0001"/>
-        </inertial>
-    </link>
-    <joint name="caster_wheel_right_joint" type="revolute">
-        <parent link="base_link"/>
-        <child link="caster_wheel_right"/>
-        <axis xyz="1 0 0"/>
-        <origin rpy="0 0 0" xyz="-4.75 -2.275 0.65"/>
-        <limit lower="-1.57" upper="1.57" effort="30.0" velocity="10.0"/>
-    </joint>
-    <link name="driver_wheel_right">
-        <visual>
-            <origin rpy="0 0 0" xyz="0 0 0"/>
-            <geometry>
-                <mesh filename="package://robot_description/meshes/wheel_right_side.stl" scale="0.01 0.01 0.01"/>
-            </geometry>
-        </visual>
-        <collision>
-            <origin rpy="0 0 0" xyz="0 0 0"/>
-            <geometry>
-                <mesh filename="package://robot_description/meshes/wheel_right_side.stl" scale="0.01 0.01 0.01"/>
-            </geometry>
-        </collision>
-        <inertial>
-            <origin xyz="0 0 0" rpy="0 0 0"/>
-            <mass value="0.3"/> <!-- kg -->
-            <inertia ixx="0.0002" ixy="0" ixz="0" iyy="0.0002" iyz="0" izz="0.0001"/>
-        </inertial>
-    </link>
-    <joint name="driver_wheel_right_joint" type="revolute">
-        <parent link="base_link"/>
-        <child link="driver_wheel_right"/>
-        <axis xyz="1 0 0"/>
-        <origin rpy="0 0 0" xyz="-4.75 2.275 0.65"/>
-        <limit lower="-1.57" upper="1.57" effort="30.0" velocity="10.0"/>
-    </joint>
-    <link name="driver_wheel_left">
-        <visual>
-            <origin rpy="0 0 0" xyz="0 0 0"/>
-            <geometry>
-                <mesh filename="package://robot_description/meshes/wheel_left_side.stl" scale="0.01 0.01 0.01"/>
-            </geometry>
-        </visual>
-        <collision>
-            <origin rpy="0 0 0" xyz="0 0 0"/>
-            <geometry>
-                <mesh filename="package://robot_description/meshes/wheel_left_side.stl" scale="0.01 0.01 0.01"/>
-            </geometry>
-        </collision>
-        <inertial>
-            <origin xyz="0 0 0" rpy="0 0 0"/>
-            <mass value="0.3"/> <!-- kg -->
-            <inertia ixx="0.0002" ixy="0" ixz="0" iyy="0.0002" iyz="0" izz="0.0001"/>
-        </inertial>
-    </link>
-    <joint name="driver_wheel_left_joint" type="revolute">
-        <parent link="base_link"/>
-        <child link="driver_wheel_left"/>
-        <axis xyz="1 0 0"/>
-        <origin rpy="0 0 0" xyz="4.75 2.275 0.65"/>
-        <limit lower="-1.57" upper="1.57" effort="30.0" velocity="10.0"/>
-    </joint>
-    <link name="manipulator_base">
-        <visual>
-            <origin rpy="0 0 0" xyz="0 0 0"/>
-            <geometry>
-                <mesh filename="package://robot_description/meshes/Base.stl" scale="0.01 0.01 0.01"/>
-            </geometry>
-        </visual>
-        <collision>
-            <origin rpy="0 0 0" xyz="0 0 0"/>
-            <geometry>
-                <mesh filename="package://robot_description/meshes/Base.stl" scale="0.01 0.01 0.01"/>
-            </geometry>
-        </collision>
-        <inertial>
-            <origin xyz="0 0 0" rpy="0 0 0"/>
-            <mass value="3.0"/>
-            <inertia ixx="0.02" ixy="0" ixz="0" iyy="0.02" iyz="0" izz="0.03"/>
-        </inertial>
-    </link>
-    <joint name="manipulator_base_mobile_joint" type="fixed">
-        <parent link="base_link"/>
-        <child link="manipulator_base"/>
-        <origin rpy="0 0 0" xyz="0 0 1.3"/>
-    </joint>
-    <link name="manipulator_shoulder">
-        <visual>
-            <origin rpy="0 0 0" xyz="0 0 0"/>
-            <geometry>
-                <mesh filename="package://robot_description/meshes/Shoulder.stl" scale="0.01 0.01 0.01"/>
-            </geometry>
-        </visual>
-        <collision>
-            <origin rpy="0 0 0" xyz="0 0 0"/>
-            <geometry>
-                <mesh filename="package://robot_description/meshes/Shoulder.stl" scale="0.01 0.01 0.01"/>
-            </geometry>
-        </collision>
-        <inertial>
-            <origin xyz="0 0 0.1" rpy="0 0 0"/>
-            <mass value="2.0"/>
-            <inertia ixx="0.005" ixy="0" ixz="0" iyy="0.005" iyz="0" izz="0.002"/>
-        </inertial>
-    </link>
-    <joint name="manipulator_base_shoulder_joint" type="revolute">
-        <parent link="manipulator_base"/>
-        <child link="manipulator_shoulder"/>
-        <axis xyz="0 0 1"/>
-        <origin rpy="0 0 0" xyz="0 0 1.7"/>
-        <limit lower="-1.57" upper="1.57" effort="30.0" velocity="10.0"/>
-    </joint>
-    <link name="manipulator_link">
-        <visual>
-            <origin rpy="0 0 0" xyz="0 0 0"/>
-            <geometry>
-                <mesh filename="package://robot_description/meshes/Link.stl" scale="0.01 0.01 0.01"/>
-            </geometry>
-        </visual>
-        <collision>
-            <origin rpy="0 0 0" xyz="0 0 0"/>
-            <geometry>
-                <mesh filename="package://robot_description/meshes/Link.stl" scale="0.01 0.01 0.01"/>
-            </geometry>
-        </collision>
-        <inertial>
-            <origin xyz="0 0 0.15" rpy="0 0 0"/>
-            <mass value="1.5"/>
-            <inertia ixx="0.003" ixy="0" ixz="0" iyy="0.003" iyz="0" izz="0.001"/>
-        </inertial>
-    </link>
-    <joint name="manipulator_shoulder_link_joint" type="revolute">
-        <parent link="manipulator_shoulder"/>
-        <child link="manipulator_link"/>
-        <axis xyz="1 0 0"/>
-        <origin rpy="0 0 0" xyz="0 0 3.36"/>
-        <limit lower="-1.57" upper="1.57" effort="30.0" velocity="10.0"/>
-    </joint>
-    <link name="manipulator_elbow">
-        <visual>
-            <origin rpy="0 0 0" xyz="0 0 0"/>
-            <geometry>
-                <mesh filename="package://robot_description/meshes/Elbow.stl" scale="0.01 0.01 0.01"/>
-            </geometry>
-        </visual>
-        <collision>
-            <origin rpy="0 0 0" xyz="0 0 0"/>
-            <geometry>
-                <mesh filename="package://robot_description/meshes/Elbow.stl" scale="0.01 0.01 0.01"/>
-            </geometry>
-        </collision>
-        <inertial>
-            <origin xyz="0 0 0.05" rpy="0 0 0"/>
-            <mass value="1.0"/>
-            <inertia ixx="0.002" ixy="0" ixz="0" iyy="0.002" iyz="0" izz="0.001"/>
-        </inertial>
-    </link>
-    <joint name="manipulator_link_elbow_joint" type="revolute">
-        <parent link="manipulator_link"/>
-        <child link="manipulator_elbow"/>
-        <axis xyz="1 0 0"/>
-        <origin rpy="0 0 0" xyz="0 0 5"/>
-        <limit lower="-1.57" upper="1.57" effort="30.0" velocity="10.0"/>
-    </joint>
-    <link name="manipulator_wrist">
-        <visual>
-            <origin rpy="0 0 0" xyz="0 0 0"/>
-            <geometry>
-                <mesh filename="package://robot_description/meshes/Wrist.stl" scale="0.01 0.01 0.01"/>
-            </geometry>
-        </visual>
-        <collision>
-            <origin rpy="0 0 0" xyz="0 0 0"/>
-            <geometry>
-                <mesh filename="package://robot_description/meshes/Wrist.stl" scale="0.01 0.01 0.01"/>
-            </geometry>
-        </collision>
-        <inertial>
-            <origin xyz="0 0 0.03" rpy="0 0 0"/>
-            <mass value="0.8"/>
-            <inertia ixx="0.0008" ixy="0" ixz="0" iyy="0.0008" iyz="0" izz="0.0005"/>
-        </inertial>
-    </link>
-    <joint name="manipulator_elbow_wrist_joint" type="revolute">
-        <parent link="manipulator_elbow"/>
-        <child link="manipulator_wrist"/>
-        <axis xyz="1 0 0"/>
-        <origin rpy="0 0 0" xyz="0 -4.27455 1.45"/>
-        <limit lower="-1.57" upper="1.57" effort="30.0" velocity="10.0"/>
-    </joint>
-    <link name="manipulator_gripper">
-        <visual>
-            <origin rpy="0 0 0" xyz="0 0 0"/>
-            <geometry>
-                <mesh filename="package://robot_description/meshes/Gripper.stl" scale="0.01 0.01 0.01"/>
-            </geometry>
-        </visual>
-        <collision>
-            <origin rpy="0 0 0" xyz="0 0 0"/>
-            <geometry>
-                <mesh filename="package://robot_description/meshes/Gripper.stl" scale="0.01 0.01 0.01"/>
-            </geometry>
-        </collision>
-        <inertial>
-            <origin xyz="0 0 0.02" rpy="0 0 0"/>
-            <mass value="0.5"/>
-            <inertia ixx="0.0005" ixy="0" ixz="0" iyy="0.0005" iyz="0" izz="0.0003"/>
-        </inertial>
-    </link>
-    <joint name="manipulator_wrist_gripper_joint" type="revolute">
-        <parent link="manipulator_wrist"/>
-        <child link="manipulator_gripper"/>
-        <axis xyz="0 1 0"/>
-        <origin rpy="0 0 0" xyz="0 -1.05 0"/>
-        <limit lower="-1.57" upper="1.57" effort="30.0" velocity="10.0"/>
-    </joint>
+<robot name="Robot" xmlns:xacro="http://ros.org/wiki/xacro">
+    <xacro:include filename="$(find robot_description)/urdf/gazebo.xacro"/>
+    <xacro:include filename="$(find robot_description)/urdf/ros2_control.xacro"/>
+    <xacro:include filename="$(find robot_description)/urdf/transmission.xacro"/>]
+    <xacro:include filename="$(find robot_description)/urdf/links.xacro"/>
+    <xacro:include filename="$(find robot_description)/urdf/joints.xacro"/>
 </robot>
